File: Breadboad-10V-Pot-board.sch (KiCad schematic (older format))
At the start: 27 parts, among them P1 DIP14, P2 DIP14, U1 TL072-, U2 TL072-, U3 TL072-

Commit message: added jack board and laid out mechanical holes for panel separation
Parts:
- added J1, J2: JACK_MONO_SW, symbol JACK_MONO_SW
- added P3: DIP_6, symbol DIP_6
Connections:
- net GND: now also J1.1, J2.1, P3.2 (P2), P3.5 (P5)
- new net JACK1: J1.3, P3.1 (P1), P3.6 (P6)
- new net JACK2: J2.3, P3.3 (P3), P3.4 (P4)
- no-connect marks 0 -> 2
Changed lines of the file:
@@
 LIBS:MySynthParts
 LIBS:Breadboad-10V-Pot-board-cache
-EELAYER 25 0
+EELAYER 24 0
 EELAYER END
 $Descr A4 11693 8268
@@
 	7550 5450 7550 4550
 Connection ~ 7550 4550
+$Comp
+L JACK_MONO_SW J1
+U 1 1 55288442
+P 5350 4900
+F 0 "J1" H 4800 4800 60  0000 C CNN
+F 1 "JACK_MONO_SW" H 5100 5100 60  0000 C CNN
+F 2 "" H 5250 4900 60  0000 C CNN
+F 3 "" H 5250 4900 60  0000 C CNN
+	1    5350 4900
+	1    0    0    -1
+$EndComp
+$Comp
+L JACK_MONO_SW J2
+U 1 1 5528865E
+P 5350 5450
+F 0 "J2" H 4800 5350 60  0000 C CNN
+F 1 "JACK_MONO_SW" H 5100 5650 60  0000 C CNN
+F 2 "" H 5250 5450 60  0000 C CNN
+F 3 "" H 5250 5450 60  0000 C CNN
+	1    5350 5450
+	1    0    0    -1
+$EndComp
+NoConn ~ 5600 4900
+NoConn ~ 5600 5450
+$Comp
+L GND_E #PWR037
+U 1 1 552886A0
+P 6250 5450
+F 0 "#PWR037" V 6250 5450 30  0001 C CNN
+F 1 "GND_E" H 6250 5380 30  0001 C CNN
+F 2 "" H 6250 5450 60  0000 C CNN
+F 3 "" H 6250 5450 60  0000 C CNN
+	1    6250 5450
+	1    0    0    -1
+$EndComp
+Wire Wire Line
+	5600 5300 6250 5300
+Wire Wire Line
+	6250 5300 6250 5450
+$Comp
+L GND_E #PWR038
+U 1 1 5528876F
+P 6250 4900
+F 0 "#PWR038" V 6250 4900 30  0001 C CNN
+F 1 "GND_E" H 6250 4830 30  0001 C CNN
+F 2 "" H 6250 4900 60  0000 C CNN
+F 3 "" H 6250 4900 60  0000 C CNN
+	1    6250 4900
+	1    0    0    -1
+$EndComp
+Wire Wire Line
+	5600 4750 6250 4750
+Wire Wire Line
+	6250 4750 6250 4900
+Text GLabel 5600 5050 2    60   BiDi ~ 0
+JACK1
+Text GLabel 5600 5600 2    60   BiDi ~ 0
+JACK2
+$Comp
+L DIP_6 P3
+U 1 1 5528909E
+P 5700 6050
+F 0 "P3" H 5700 6250 50  0000 C CNN
+F 1 "DIP_6" H 5700 5850 50  0000 C CNN
+F 2 "" H 5700 4850 60  0000 C CNN
+F 3 "" H 5700 4850 60  0000 C CNN
+	1    5700 6050
+	1    0    0    -1
+$EndComp
+Text GLabel 5950 5950 2    60   BiDi ~ 0
+JACK1
+Text GLabel 5450 5950 0    60   BiDi ~ 0
+JACK1
+Text GLabel 5450 6150 0    60   BiDi ~ 0
+JACK2
+Text GLabel 5950 6150 2    60   BiDi ~ 0
+JACK2
+$Comp
+L GND_E #PWR039
+U 1 1 5528921B
+P 6600 6200
+F 0 "#PWR039" V 6600 6200 30  0001 C CNN
+F 1 "GND_E" H 6600 6130 30  0001 C CNN
+F 2 "" H 6600 6200 60  0000 C CNN
+F 3 "" H 6600 6200 60  0000 C CNN
+	1    6600 6200
+	1    0    0    -1
+$EndComp
+Wire Wire Line
+	5950 6050 6600 6050
+Wire Wire Line
+	6600 6050 6600 6200
+$Comp
+L GND_E #PWR040
+U 1 1 55289265
+P 4800 6200
+F 0 "#PWR040" V 4800 6200 30  0001 C CNN
+F 1 "GND_E" H 4800 6130 30  0001 C CNN
+F 2 "" H 4800 6200 60  0000 C CNN
+F 3 "" H 4800 6200 60  0000 C CNN
+	1    4800 6200
+	-1   0    0    -1
+$EndComp
+Wire Wire Line
+	5450 6050 4800 6050
+Wire Wire Line
+	4800 6050 4800 6200
 $EndSCHEMATC
